File: hardware/GateDrive.kicad_sch (KiCad schematic)
At the start: 0 parts

Commit message: Populate Gate Drive sheet (DRV8323R), fix MCU Core PWM pin gap
- DRV8323RSRGZT (=DRV8323R) fully wired per the real TI datasheet
  (SLVSDJ3D, fetched directly): single shared charge pump (not
  per-phase bootstrap caps as originally assumed), VDD/DVDD internal
  LDO decoupling only, VREF self-referenced, optional 600mA buck
  disabled (nSHD tied to GND), CAL tied to GND
- Caught and fixed a real gap before it became a wiring mistake: the
  chip needs 6 direct hardware PWM pins (INHA/INLA/INHB/INLB/INHC/
  INLC) in addition to SPI - missed in the first pass. Also removed a
  fictitious 'nSLEEP' pin that doesn't exist on this part (ENABLE
  alone controls sleep). Reassigned MCU Core GPIOs accordingly and
  added 10k pull-downs on all 6 PWM inputs + ENABLE for a safe
  power-up default (gates off until firmware takes over)
- ARCHITECTURE.md updated with corrected pin map and rationale

Co-Authored-By: Claude Sonnet 5 <noreply@anthropic.com>
Parts:
- added C23: CP flying cap, symbol METUPowerLab_Capacitors_Ceramics_SurfaceMounts:47 nF 100V
- added C24: VCP decouple, symbol METUPowerLab_Capacitors_Ceramics_SurfaceMounts:1 µF
- added C25: VM hf decouple, symbol METUPowerLab_Capacitors_Ceramics_SurfaceMounts:100 nF
- added C26: VM bulk decouple, symbol METUPowerLab_Capacitors_Ceramics_SurfaceMounts:10 µF 75V
- added C27: DVDD decouple, symbol METUPowerLab_Capacitors_Ceramics_SurfaceMounts:1 µF
- added C28: VREF decouple, symbol METUPowerLab_Capacitors_Ceramics_SurfaceMounts:100 nF
- added R16: INHA pulldown, symbol METUPowerLab_Resistors_ChipResistors:10 kOhm
- added R17: INLA pulldown, symbol METUPowerLab_Resistors_ChipResistors:10 kOhm
- added R18: INHB pulldown, symbol METUPowerLab_Resistors_ChipResistors:10 kOhm
- added R19: INLB pulldown, symbol METUPowerLab_Resistors_ChipResistors:10 kOhm
- added R20: INHC pulldown, symbol METUPowerLab_Resistors_ChipResistors:10 kOhm
- added R21: INLC pulldown, symbol METUPowerLab_Resistors_ChipResistors:10 kOhm
- added R22: ENABLE pulldown, symbol METUPowerLab_Resistors_ChipResistors:10 kOhm
- added R23: SDO pullup, symbol METUPowerLab_Resistors_ChipResistors:10 kOhm
- added U6: DRV8323RSRGZT, METUPowerLab_MotorDrivers_BLDC:48-VQFN, symbol METUPowerLab_MotorDrivers_BLDC:DRV8323RSRGZT
Connections:
- new net +3V3_MCU: R23.2
- new net +VBUS_PROT: C24.2, C25.1, C26.1, U6.6 (VM), U6.7 (VDRAIN)
- new net CP_CPH: C23.1, U6.4 (CPH)
- new net CP_CPL: C23.2, U6.3 (CPL)
- new net CP_VCP: C24.1, U6.5 (VCP)
- new net DVDD_DECOUPLE: C27.1, U6.36 (DVDD)
- new net ENABLE: R22.1, U6.33 (ENABLE)
- new net GHA: U6.8 (GHA)
- new net GHB: U6.17 (GHB)
- new net GHC: U6.18 (GHC)
- new net GLA: U6.10 (GLA)
- new net GLB: U6.15 (GLB)
- new net GLC: U6.20 (GLC)
- new net GND: C25.2, C26.2, C27.2, C28.2, R16.1, R16.2, R17.2, R18.2, R19.2, R20.2, R21.2, R22.2, U6.2 (PGND), U6.27 (DGND), U6.34 (CAL), U6.35 (AGND), U6.37 (INHA), U6.43 (BGND), U6.48 (nSHD), U6.Shield
- new net INHB: R18.1, U6.39 (INHB)
- new net INHC: R20.1, U6.41 (INHC)
- new net INLA: R17.1, U6.38 (INLA)
- new net INLB: R19.1, U6.40 (INLB)
- new net INLC: R21.1, U6.42 (INLC)
- new net SCLK: U6.31 (SCLK)
- new net SDI: U6.30 (SDI)
- new net SDO: R23.1, U6.29 (SDO)
- new net SHA: U6.9 (SHA)
- new net SHB: U6.16 (SHB)
- new net SHC: U6.19 (SHC)
- new net SNA: U6.12 (SNA)
- new net SNB: U6.13 (SNB)
- new net SNC: U6.22 (SNC)
- new net SOA: U6.25 (SOA)
- new net SOB: U6.24 (SOB)
- new net SOC: U6.23 (SOC)
- new net SPA: U6.11 (SPA)
- new net SPB: U6.14 (SPB)
- new net SPC: U6.21 (SPC)
- new net VREF_DECOUPLE: C28.1, U6.26 (VREF)
- new net nFAULT: U6.28 (nFAULT)
- new net nSCS: U6.32 (nSCS)
- no-connect marks 0 -> 5
Other:
- note added: "LAYOUT: Place C23 (charge pump cap) and C24 (VCP decouple) as close as possible to U6 pins 3/4/5 LAYOUT: Place C25/C26 (VM decoupling) directly across U6 VM/PGND pins, shortest loop LAYOUT: Keep CP_CPH/CP_CPL/CP_VCP traces short, away from switching nodes (GHx/SHx/GLx)"

Commit message: Populate Current Sensing + Communication sheets; schematic complete
Current Sensing:
- DC-bus shunt (5 mOhm, in series after the eFuse - required renaming
  the eFuse OUT net to +VBUS_EFUSE_OUT so the shunt sits properly
  in-line ahead of +VBUS_PROT)
- INA240 total-bus current sense, unidirectional config, -> MCU ADC

Communication:
- SN65HVD230 CAN transceiver (3.3V native) on ESP32 TWAI pins
- Per-line TVS (SP0115-01UTG) on CANH/CANL
- 4-pin bus connector (CANH/CANL/GND/+VBUS_PROT)

Whole-hierarchy ERC (all 6 sheets + root) now down to 3 residual
errors, all the same benign/expected 'two power_out pins on one net'
pattern (datasheet-recommended parallel pins, or a PWR_FLAG sharing
a net with a real driver) - fully explained in ARCHITECTURE.md, which
now also documents the found-and-worked-around vendor library defects
(eFuse pin-20 duplication, TMP235 VOUT mistyped as input) and confirms
the shunt 'duplicate pins' are correct 4-terminal Kelvin modeling, not
a bug.

All 6 hierarchical sheets are now fully wired end to end:
Power Supply -> MCU Core -> Gate Drive -> Power Stage, with Current
Sensing and Communication cross-wired throughout.

Co-Authored-By: Claude Sonnet 5 <noreply@anthropic.com>
Changed lines of the file:
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@@
+		)
+	)
+	(symbol
+		(lib_id "power:PWR_FLAG")
+		(at 177.8 52.07 0)
+		(unit 1)
+		(body_style 1)
+		(exclude_from_sim no)
+		(in_bom yes)
+		(on_board yes)
+		(in_pos_files yes)
+		(dnp no)
+		(property "Reference" "#FLG8"
+			(at 177.8 53.975 0)
+			(hide yes)
+			(show_name no)
+			(do_not_autoplace no)
+			(effects
+				(font
+					(size 1.27 1.27)
+				)
+			)
+		)
+		(property "Value" "PWR_FLAG"
+			(at 177.8 55.88 0)
+			(show_name no)
+			(do_not_autoplace no)
+			(effects
+				(font
+					(size 1.27 1.27)
+				)
+			)
+		)
+		(property "Footprint" ""
+			(at 177.8 52.07 0)
+			(hide yes)
+			(show_name no)
+			(do_not_autoplace no)
+			(effects
+				(font
+					(size 1.27 1.27)
+				)
+			)
+		)
+		(property "Datasheet" ""
+			(at 177.8 52.07 0)
+			(hide yes)
+			(show_name no)
+			(do_not_autoplace no)
+			(effects
+				(font
+					(size 1.27 1.27)
+				)
+			)
+		)
+		(property "Description" "Special symbol for telling ERC where power comes from"
+			(at 177.8 52.07 0)
+			(hide yes)
+			(show_name no)
+			(do_not_autoplace no)
+			(effects
+				(font
+					(size 1.27 1.27)
+				)
+			)
+		)
+		(pin "1"
+		)
+		(instances
+			(project "ESC3Phase"
+				(path "/e28ad77e-eee8-4da9-a82f-57fba8403d74"
+					(reference "#FLG8")
+					(unit 1)
+				)
+			)
+		)
+	)
+	(label "VREF_DECOUPLE"
+		(at 177.8 52.07 270)
+		(effects
+			(font
+				(size 1.27 1.27)
+			)
+			(justify right bottom)
 		)
 	)

Commit message: PCB layout: board outline, mounting holes, footprint placement, copper pours, phase-output routing
- 100x115mm 2-layer board, 4x M3 mounting holes, design rules per PowerLab spec
- All 55 schematic components synced to board with real footprints
- Auto-placed via force-directed placement with locked connector/MCU anchors
- GND pour (both layers) + localized pours for VIN_RAW/+VBUS/+VBUS_EFUSE_OUT/+VBUS_PROT/+5V_LOGIC
- Routed the 3 critical phase-output traces (SHA/SHB/SHC, 2mm wide)
- Documented full PCB status in ARCHITECTURE.md: NOT yet fab-ready (732 DRC
  violations, 21 courtyard overlaps, ~50 signal nets still unrouted since
  Freerouting is unavailable in this environment)

Co-Authored-By: Claude Sonnet 5 <noreply@anthropic.com>
Parts:
- C23: footprint (none) -> METUPowerLab_Capacitors_Ceramics_SurfaceMounts:0805_Medium
- C24, C25, C27, C28: footprint (none) -> METUPowerLab_Capacitors_Ceramics_SurfaceMounts:0603_Medium
- C26: footprint (none) -> METUPowerLab_Capacitors_Ceramics_SurfaceMounts:2220
- R16, R17, R18, R19, R20, R21, R22, R23: footprint (none) -> METUPowerLab_Resistors_ChipResistors:0603_Medium
Changed lines of the file:
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@@
 			)
 		)
-		(property "Footprint" ""
+		(property "Footprint" "METUPowerLab_Capacitors_Ceramics_SurfaceMounts:0805_Medium"
 			(at 101.295 21.59 0)
 			(hide yes)
@@
 			)
 		)
-		(property "Footprint" ""
+		(property "Footprint" "METUPowerLab_Capacitors_Ceramics_SurfaceMounts:0603_Medium"
 			(at 101.295 2.54 0)
 			(hide yes)
@@
 			)
 		)
-		(property "Footprint" ""
+		(property "Footprint" "METUPowerLab_Capacitors_Ceramics_SurfaceMounts:0603_Medium"
 			(at 101.295 -5.08 0)
 			(hide yes)
@@
 			)
 		)
-		(property "Footprint" ""
+		(property "Footprint" "METUPowerLab_Capacitors_Ceramics_SurfaceMounts:2220"
 			(at 92.405 -5.08 0)
 			(hide yes)
@@
 			)
 		)
-		(property "Footprint" ""
+		(property "Footprint" "METUPowerLab_Capacitors_Ceramics_SurfaceMounts:0603_Medium"
 			(at 101.295 30.48 0)
 			(hide yes)
@@
 			)
 		)
-		(property "Footprint" ""
+		(property "Footprint" "METUPowerLab_Capacitors_Ceramics_SurfaceMounts:0603_Medium"
 			(at 186.385 48.26 0)
 			(hide yes)
@@
 			)
 		)
-		(property "Footprint" ""
+		(property "Footprint" "METUPowerLab_Resistors_ChipResistors:0603_Medium"
 			(at 106.426 39.116 90)
 			(hide yes)
@@
 			)
 		)
-		(property "Footprint" ""
+		(property "Footprint" "METUPowerLab_Resistors_ChipResistors:0603_Medium"
 			(at 106.426 41.656 90)
 			(hide yes)
@@
 			)
 		)
-		(property "Footprint" ""
+		(property "Footprint" "METUPowerLab_Resistors_ChipResistors:0603_Medium"
 			(at 106.426 46.736 90)
 			(hide yes)
@@
 			)
 		)
-		(property "Footprint" ""
+		(property "Footprint" "METUPowerLab_Resistors_ChipResistors:0603_Medium"
 			(at 106.426 49.276 90)
 			(hide yes)
@@
 			)
 		)
-		(property "Footprint" ""
+		(property "Footprint" "METUPowerLab_Resistors_ChipResistors:0603_Medium"
 			(at 106.426 54.356 90)
 			(hide yes)
@@
 			)
 		)
-		(property "Footprint" ""
+		(property "Footprint" "METUPowerLab_Resistors_ChipResistors:0603_Medium"
 			(at 106.426 58.166 90)
 			(hide yes)
@@
 			)
 		)
-		(property "Footprint" ""
+		(property "Footprint" "METUPowerLab_Resistors_ChipResistors:0603_Medium"
 			(at 106.426 16.256 90)
 			(hide yes)
@@
 			)
 		)
-		(property "Footprint" ""
+		(property "Footprint" "METUPowerLab_Resistors_ChipResistors:0603_Medium"
 			(at 106.426 64.516 90)
 			(hide yes)
